Commit message: add collision meshes

File: urdf/abb_irb4600_40_255_macro.xacro (robot description, xacro)
@@ -4,23 +4,38 @@
         <!-- link list -->
         <link name="${prefix}base_link">
-            <visual name="visual">
+            <visual>
                 <geometry>
                     <mesh filename="package://abb_irb4600_description/meshes/visual/base_link.dae"/>
                 </geometry>
             </visual>
+            <collision>
+                <geometry>
+                    <mesh filename="package://abb_irb4600_description/meshes/collision/base_link_collision.stl"/>
+                </geometry>
+            </collision>
         </link>
         <link name="${prefix}link_1">
-            <visual name="visual">
+            <visual>
                 <geometry>
                     <mesh filename="package://abb_irb4600_description/meshes/visual/link1.dae"/>
                 </geometry>
             </visual>
+            <collision>
+                <geometry>
+                    <mesh filename="package://abb_irb4600_description/meshes/collision/link1_collision.stl"/>
+                </geometry>
+            </collision>
         </link>
         <link name="${prefix}link_2">
-            <visual name="visual">
+            <visual>
                 <geometry>
                     <mesh filename="package://abb_irb4600_description/meshes/visual/link2.dae"/>
                 </geometry>
             </visual>
+            <collision>
+                <geometry>
+                    <mesh filename="package://abb_irb4600_description/meshes/collision/link2_collision.stl"/>
+                </geometry>
+            </collision>
         </link>
         <link name="${prefix}link_3">
@@ -30,4 +45,9 @@
                 </geometry>
             </visual>
+            <collision>
+                <geometry>
+                    <mesh filename="package://abb_irb4600_description/meshes/collision/link3_collision.stl"/>
+                </geometry>
+            </collision>
         </link>
         <link name="${prefix}link_4">
@@ -37,4 +57,9 @@
                 </geometry>
             </visual>
+            <collision>
+                <geometry>
+                    <mesh filename="package://abb_irb4600_description/meshes/collision/link4_collision.stl"/>
+                </geometry>
+            </collision>
         </link>
         <link name="${prefix}link_5">
@@ -44,4 +69,9 @@
                 </geometry>
             </visual>
+            <collision>
+                <geometry>
+                    <mesh filename="package://abb_irb4600_description/meshes/collision/link5_collision.stl"/>
+                </geometry>
+            </collision>
         </link>
         <link name="${prefix}link_6">
@@ -51,4 +81,9 @@
                 </geometry>
             </visual>
+            <collision>
+                <geometry>
+                    <mesh filename="package://abb_irb4600_description/meshes/collision/link6_collision.stl"/>
+                </geometry>
+            </collision>
         </link>
         <!-- end of link list-->

Commit message: edit urdf to make ik_fast solutions faster

File: urdf/abb_irb4600_40_255_macro.xacro (robot description, xacro)
@@ -97,6 +97,6 @@
         </joint>
         <joint type="revolute" name="${prefix}joint_2">
-            <origin xyz="0.175 0 0" rpy="${radians(-90)} ${radians(-90)} 0"/>
-            <axis xyz="0 0 1"/>
+            <origin xyz="0.175 0 0" rpy="0 0 0"/>
+            <axis xyz="0 1 0"/>
             <parent link="${prefix}link_1"/>
             <child link="${prefix}link_2"/>
@@ -104,6 +104,6 @@
         </joint>
         <joint type="revolute" name="${prefix}joint_3">
-            <origin xyz="1.095 0 0" rpy="0 0 0"/>
-            <axis xyz="0 0 1"/>
+            <origin xyz="0 0 1.095" rpy="0 0 0"/>
+            <axis xyz="0 1 0"/>
             <parent link="${prefix}link_2"/>
             <child link="${prefix}link_3"/>
@@ -111,6 +111,6 @@
         </joint>
         <joint type="revolute" name="${prefix}joint_4">
-            <origin xyz="0.175 0.3306 0" rpy="${radians(-90)} 0 0"/>
-            <axis xyz="0 0 1"/>
+            <origin xyz="0 0 0.175" rpy="0 0 0"/>
+            <axis xyz="1 0 0"/>
             <parent link="${prefix}link_3"/>
             <child link="${prefix}link_4"/>
@@ -118,6 +118,6 @@
         </joint>
         <joint type="revolute" name="${prefix}joint_5">
-            <origin xyz="0 0 0.9385" rpy="${radians(-90)} 0 0"/>
-            <axis xyz="0 0 1"/>
+            <origin xyz="1.270 0 0" rpy="0 0 0"/>
+            <axis xyz="0 1 0"/>
             <parent link="${prefix}link_4"/>
             <child link="${prefix}link_5"/>
@@ -125,6 +125,6 @@
         </joint>
         <joint type="revolute" name="${prefix}joint_6">
-            <origin xyz="0 0 0" rpy="${radians(90)} 0 0"/>
-            <axis xyz="0 0 1"/>
+            <origin xyz="0 0 0" rpy="0 0 0"/>
+            <axis xyz="1 0 0"/>
             <parent link="${prefix}link_5"/>
             <child link="${prefix}link_6"/>
@@ -142,5 +142,5 @@
         <link name="${prefix}flange"/>
         <joint type="fixed" name="${prefix}joint_6-flange">
-            <origin xyz="0 0 0.135" rpy="0 0 0"/>
+            <origin xyz="0.135 0 0" rpy="0 0 0"/>
             <parent link="${prefix}link_6"/>
             <child link="${prefix}flange"/>
