Commit message: clean up package

File: urdf/abb_irb4600_40_255.xacro (robot description, xacro)
@@ -1,5 +1,14 @@
 <?xml version="1.0" ?>
 <robot name="abb_irb4600_40_255" xmlns:xacro="http://ros.org/wiki/xacro">
+  <xacro:arg name="prefix" default=""/>
   <xacro:include filename="$(find abb_irb4600_description)/urdf/abb_irb4600_40_255_macro.xacro"/>
-  <xacro:abb_irb4600_40_255 prefix=""/>
+  <xacro:abb_irb4600_40_255 prefix="$(arg prefix)"/>
+  <!-- 'world' frame: default pose reference frame -->
+  <link name="world" />
+  <joint name="world-$(arg prefix)base_link" type="fixed">
+    <origin xyz="0 0 0" rpy="0 0 0"/>
+    <axis xyz="0 0 1"/>
+    <parent link="world"/>
+    <child link="$(arg prefix)base_link"/>
+  </joint>
 </robot>

File: urdf/abb_irb4600_40_255_macro.xacro (robot description, xacro)
@@ -1,156 +1,156 @@
 <?xml version="1.0"?>
 <robot xmlns:xacro="http://ros.org/wiki/xacro">
-    <xacro:macro name="abb_irb4600_40_255" params="prefix">
-        <!-- link list -->
-        <link name="${prefix}base_link">
-            <visual>
-                <geometry>
-                    <mesh filename="package://abb_irb4600_description/meshes/visual/base_link.dae"/>
-                </geometry>
-            </visual>
-            <collision>
-                <geometry>
-                    <mesh filename="package://abb_irb4600_description/meshes/collision/base_link_collision.stl"/>
-                </geometry>
-            </collision>
-        </link>
-        <link name="${prefix}link_1">
-            <visual>
-                <geometry>
-                    <mesh filename="package://abb_irb4600_description/meshes/visual/link1.dae"/>
-                </geometry>
-            </visual>
-            <collision>
-                <geometry>
-                    <mesh filename="package://abb_irb4600_description/meshes/collision/link1_collision.stl"/>
-                </geometry>
-            </collision>
-        </link>
-        <link name="${prefix}link_2">
-            <visual>
-                <geometry>
-                    <mesh filename="package://abb_irb4600_description/meshes/visual/link2.dae"/>
-                </geometry>
-            </visual>
-            <collision>
-                <geometry>
-                    <mesh filename="package://abb_irb4600_description/meshes/collision/link2_collision.stl"/>
-                </geometry>
-            </collision>
-        </link>
-        <link name="${prefix}link_3">
-            <visual name="visual">
-                <geometry>
-                    <mesh filename="package://abb_irb4600_description/meshes/visual/link3.dae"/>
-                </geometry>
-            </visual>
-            <collision>
-                <geometry>
-                    <mesh filename="package://abb_irb4600_description/meshes/collision/link3_collision.stl"/>
-                </geometry>
-            </collision>
-        </link>
-        <link name="${prefix}link_4">
-            <visual name="visual">
-                <geometry>
-                    <mesh filename="package://abb_irb4600_description/meshes/visual/link4.dae"/>
-                </geometry>
-            </visual>
-            <collision>
-                <geometry>
-                    <mesh filename="package://abb_irb4600_description/meshes/collision/link4_collision.stl"/>
-                </geometry>
-            </collision>
-        </link>
-        <link name="${prefix}link_5">
-            <visual name="visual">
-                <geometry>
-                    <mesh filename="package://abb_irb4600_description/meshes/visual/link5.dae"/>
-                </geometry>
-            </visual>
-            <collision>
-                <geometry>
-                    <mesh filename="package://abb_irb4600_description/meshes/collision/link5_collision.stl"/>
-                </geometry>
-            </collision>
-        </link>
-        <link name="${prefix}link_6">
-            <visual name="visual">
-                <geometry>
-                    <mesh filename="package://abb_irb4600_description/meshes/visual/link6.dae"/>
-                </geometry>
-            </visual>
-            <collision>
-                <geometry>
-                    <mesh filename="package://abb_irb4600_description/meshes/collision/link6_collision.stl"/>
-                </geometry>
-            </collision>
-        </link>
-        <!-- end of link list-->
-        <!-- joint list -->
-        <joint type="revolute" name="${prefix}joint_1">
-            <origin xyz="0 0 0.495" rpy="0 0 0"/>
-            <axis xyz="0 0 1"/>
-            <parent link="${prefix}base_link"/>
-            <child link="${prefix}link_1"/>
-            <limit effort="0" lower="${radians(-180)}" upper="${radians(180)}" velocity="${radians(175)}"/>
-        </joint>
-        <joint type="revolute" name="${prefix}joint_2">
-            <origin xyz="0.175 0 0" rpy="0 0 0"/>
-            <axis xyz="0 1 0"/>
-            <parent link="${prefix}link_1"/>
-            <child link="${prefix}link_2"/>
-            <limit effort="0" lower="${radians(-90)}" upper="${radians(150)}" velocity="${radians(175)}"/>
-        </joint>
-        <joint type="revolute" name="${prefix}joint_3">
-            <origin xyz="0 0 1.095" rpy="0 0 0"/>
-            <axis xyz="0 1 0"/>
-            <parent link="${prefix}link_2"/>
-            <child link="${prefix}link_3"/>
-            <limit effort="0" lower="${radians(-180)}" upper="${radians(75)}" velocity="${radians(175)}"/>
-        </joint>
-        <joint type="revolute" name="${prefix}joint_4">
-            <origin xyz="0 0 0.175" rpy="0 0 0"/>
-            <axis xyz="1 0 0"/>
-            <parent link="${prefix}link_3"/>
-            <child link="${prefix}link_4"/>
-            <limit effort="0" lower="${radians(-400)}" upper="${radians(400)}" velocity="${radians(250)}"/>
-        </joint>
-        <joint type="revolute" name="${prefix}joint_5">
-            <origin xyz="1.270 0 0" rpy="0 0 0"/>
-            <axis xyz="0 1 0"/>
-            <parent link="${prefix}link_4"/>
-            <child link="${prefix}link_5"/>
-            <limit effort="0" lower="${radians(-125)}" upper="${radians(120)}" velocity="${radians(250)}"/>
-        </joint>
-        <joint type="revolute" name="${prefix}joint_6">
-            <origin xyz="0 0 0" rpy="0 0 0"/>
-            <axis xyz="1 0 0"/>
-            <parent link="${prefix}link_5"/>
-            <child link="${prefix}link_6"/>
-            <limit effort="0" lower="${radians(-400)}" upper="${radians(400)}" velocity="${radians(360)}"/>
-        </joint>
-        <!-- end of joint list -->
-        <!-- 'base' frame: base_link to ABB World Coordinates transform  -->
-        <link name="${prefix}base" />
-        <joint name="${prefix}base_link-base" type="fixed">
-            <origin xyz="0 0 0" rpy="0 0 0"/>
-            <child link="${prefix}base_link"/>
-            <parent link="${prefix}base"/>
-        </joint>
-        <!-- ROS-Industrial 'flange' frame: attachment point for EEF models -->
-        <link name="${prefix}flange"/>
-        <joint type="fixed" name="${prefix}joint_6-flange">
-            <origin xyz="0.135 0 0" rpy="0 0 0"/>
-            <parent link="${prefix}link_6"/>
-            <child link="${prefix}flange"/>
-        </joint>
-        <!-- ROS-Industrial 'tool0' frame: all-zeros tool frame -->
-        <link name="${prefix}tool0" />
-        <joint name="${prefix}link_6-tool0" type="fixed">
-            <origin xyz="0 0 0" rpy="0 ${radians(90)} 0" />
-            <parent link="${prefix}flange" />
-            <child link="${prefix}tool0" />
-        </joint>
-    </xacro:macro>
+  <xacro:macro name="abb_irb4600_40_255" params="prefix">
+    <!-- link list -->
+    <link name="${prefix}base_link">
+      <visual>
+        <geometry>
+          <mesh filename="package://abb_irb4600_description/meshes/visual/base_link.dae"/>
+        </geometry>
+      </visual>
+      <collision>
+        <geometry>
+          <mesh filename="package://abb_irb4600_description/meshes/collision/base_link_collision.stl"/>
+        </geometry>
+      </collision>
+    </link>
+    <link name="${prefix}link_1">
+      <visual>
+        <geometry>
+          <mesh filename="package://abb_irb4600_description/meshes/visual/link1.dae"/>
+        </geometry>
+      </visual>
+      <collision>
+        <geometry>
+          <mesh filename="package://abb_irb4600_description/meshes/collision/link1_collision.stl"/>
+        </geometry>
+      </collision>
+    </link>
+    <link name="${prefix}link_2">
+      <visual>
+        <geometry>
+          <mesh filename="package://abb_irb4600_description/meshes/visual/link2.dae"/>
+        </geometry>
+      </visual>
+      <collision>
+        <geometry>
+          <mesh filename="package://abb_irb4600_description/meshes/collision/link2_collision.stl"/>
+        </geometry>
+      </collision>
+    </link>
+    <link name="${prefix}link_3">
+      <visual name="visual">
+        <geometry>
+          <mesh filename="package://abb_irb4600_description/meshes/visual/link3.dae"/>
+        </geometry>
+      </visual>
+      <collision>
+        <geometry>
+          <mesh filename="package://abb_irb4600_description/meshes/collision/link3_collision.stl"/>
+        </geometry>
+      </collision>
+    </link>
+    <link name="${prefix}link_4">
+      <visual name="visual">
+        <geometry>
+          <mesh filename="package://abb_irb4600_description/meshes/visual/link4.dae"/>
+        </geometry>
+      </visual>
+      <collision>
+        <geometry>
+          <mesh filename="package://abb_irb4600_description/meshes/collision/link4_collision.stl"/>
+        </geometry>
+      </collision>
+    </link>
+    <link name="${prefix}link_5">
+      <visual name="visual">
+        <geometry>
+          <mesh filename="package://abb_irb4600_description/meshes/visual/link5.dae"/>
+        </geometry>
+      </visual>
+      <collision>
+        <geometry>
+          <mesh filename="package://abb_irb4600_description/meshes/collision/link5_collision.stl"/>
+        </geometry>
+      </collision>
+    </link>
+    <link name="${prefix}link_6">
+      <visual name="visual">
+        <geometry>
+          <mesh filename="package://abb_irb4600_description/meshes/visual/link6.dae"/>
+        </geometry>
+      </visual>
+      <collision>
+        <geometry>
+          <mesh filename="package://abb_irb4600_description/meshes/collision/link6_collision.stl"/>
+        </geometry>
+      </collision>
+    </link>
+    <!-- end of link list-->
+    <!-- joint list -->
+    <joint type="revolute" name="${prefix}joint_1">
+      <origin xyz="0 0 0.495" rpy="0 0 0"/>
+      <axis xyz="0 0 1"/>
+      <parent link="${prefix}base_link"/>
+      <child link="${prefix}link_1"/>
+      <limit effort="0" lower="${radians(-180)}" upper="${radians(180)}" velocity="${radians(175)}"/>
+    </joint>
+    <joint type="revolute" name="${prefix}joint_2">
+      <origin xyz="0.175 0 0" rpy="0 0 0"/>
+      <axis xyz="0 1 0"/>
+      <parent link="${prefix}link_1"/>
+      <child link="${prefix}link_2"/>
+      <limit effort="0" lower="${radians(-90)}" upper="${radians(150)}" velocity="${radians(175)}"/>
+    </joint>
+    <joint type="revolute" name="${prefix}joint_3">
+      <origin xyz="0 0 1.095" rpy="0 0 0"/>
+      <axis xyz="0 1 0"/>
+      <parent link="${prefix}link_2"/>
+      <child link="${prefix}link_3"/>
+      <limit effort="0" lower="${radians(-180)}" upper="${radians(75)}" velocity="${radians(175)}"/>
+    </joint>
+    <joint type="revolute" name="${prefix}joint_4">
+      <origin xyz="0 0 0.175" rpy="0 0 0"/>
+      <axis xyz="1 0 0"/>
+      <parent link="${prefix}link_3"/>
+      <child link="${prefix}link_4"/>
+      <limit effort="0" lower="${radians(-400)}" upper="${radians(400)}" velocity="${radians(250)}"/>
+    </joint>
+    <joint type="revolute" name="${prefix}joint_5">
+      <origin xyz="1.270 0 0" rpy="0 0 0"/>
+      <axis xyz="0 1 0"/>
+      <parent link="${prefix}link_4"/>
+      <child link="${prefix}link_5"/>
+      <limit effort="0" lower="${radians(-125)}" upper="${radians(120)}" velocity="${radians(250)}"/>
+    </joint>
+    <joint type="revolute" name="${prefix}joint_6">
+      <origin xyz="0 0 0" rpy="0 0 0"/>
+      <axis xyz="1 0 0"/>
+      <parent link="${prefix}link_5"/>
+      <child link="${prefix}link_6"/>
+      <limit effort="0" lower="${radians(-400)}" upper="${radians(400)}" velocity="${radians(360)}"/>
+    </joint>
+    <!-- end of joint list -->
+    <!-- 'base' frame: base_link to ABB World Coordinates transform  -->
+    <link name="${prefix}base" />
+    <joint name="${prefix}base_link-base" type="fixed">
+      <origin xyz="0 0 0" rpy="0 0 0"/>
+      <parent link="${prefix}base_link"/>
+      <child link="${prefix}base"/>
+    </joint>
+    <!-- ROS-Industrial 'flange' frame: attachment point for EEF models -->
+    <link name="${prefix}flange"/>
+    <joint type="fixed" name="${prefix}joint_6-flange">
+      <origin xyz="0.135 0 0" rpy="0 0 0"/>
+      <parent link="${prefix}link_6"/>
+      <child link="${prefix}flange"/>
+    </joint>
+    <!-- ROS-Industrial 'tool0' frame: all-zeros tool frame -->
+    <link name="${prefix}tool0" />
+    <joint name="${prefix}link_6-tool0" type="fixed">
+      <origin xyz="0 0 0" rpy="0 ${radians(90)} 0" />
+      <parent link="${prefix}flange" />
+      <child link="${prefix}tool0" />
+    </joint>
+  </xacro:macro>
 </robot>

Commit message: migrate to ros2

File: urdf/abb_irb4600_40_255.xacro (robot description, xacro)
@@ -21,7 +21,15 @@
 <robot name="abb_irb4600_40_255" xmlns:xacro="http://ros.org/wiki/xacro">
   <xacro:arg name="prefix" default=""/>
+  <xacro:arg name="use_mock_hardware" default="true"/>
+  <xacro:arg name="include_hardware" default="true"/>
+  <xacro:arg name="initial_positions_file"
+    default="$(find abb_irb4600_description)/config/initial_positions.yaml"/>
+  <xacro:arg name="joint_limits_file"
+    default="$(find abb_irb4600_description)/config/joint_limits.yaml"/>
   <xacro:include filename="$(find abb_irb4600_description)/urdf/abb_irb4600_40_255_macro.xacro"/>
-  <xacro:abb_irb4600_40_255 prefix="$(arg prefix)"/>
-  <!-- 'world' frame: default pose reference frame -->
+  <xacro:abb_irb4600_40_255 prefix="$(arg prefix)"
+    initial_positions_file="$(arg initial_positions_file)"
+    joint_limits_parameters_file="$(arg joint_limits_file)"/>
+  <!-- 'world' frame - default pose reference frame -->
   <link name="world" />
   <joint name="world-$(arg prefix)base_link" type="fixed">

File: urdf/abb_irb4600_40_255_macro.xacro (robot description, xacro)
@@ -21,5 +21,11 @@
 -->
 <robot xmlns:xacro="http://ros.org/wiki/xacro">
-  <xacro:macro name="abb_irb4600_40_255" params="prefix">
+  <xacro:macro name="abb_irb4600_40_255" params="
+    prefix
+    initial_positions_file:='$(find abb_irb4600_description)/config/initial_positions_file.yaml'
+    joint_limits_parameters_file:='$(find abb_irb4600_description)/config/joint_limits.yaml'
+  ">
+    <xacro:property name="joint_limits_parameters" value="${xacro.load_yaml(joint_limits_parameters_file)}"/>
+    <xacro:property name="joint_limits" value="${joint_limits_parameters['joint_limits']}"/>
     <!-- link list -->
     <link name="${prefix}base_link">
@@ -109,48 +115,72 @@
     <!-- end of link list -->
     <!-- joint list -->
-    <joint type="revolute" name="${prefix}joint_1">
+    <joint name="${prefix}joint_1" type="revolute">
       <origin xyz="0 0 0.495" rpy="0 0 0"/>
       <axis xyz="0 0 1"/>
       <parent link="${prefix}base_link"/>
       <child link="${prefix}link_1"/>
-      <limit effort="0" lower="${radians(-180)}" upper="${radians(180)}" velocity="${radians(175)}"/>
-    </joint>
-    <joint type="revolute" name="${prefix}joint_2">
+      <limit
+        effort="${joint_limits['joint_1']['max_effort']}"
+        lower="${joint_limits['joint_1']['min_position']}"
+        upper="${joint_limits['joint_1']['max_position']}"
+        velocity="${joint_limits['joint_1']['max_velocity']}"/>
+    </joint>
+    <joint name="${prefix}joint_2" type="revolute">
       <origin xyz="0.175 0 0" rpy="0 0 0"/>
       <axis xyz="0 1 0"/>
       <parent link="${prefix}link_1"/>
       <child link="${prefix}link_2"/>
-      <limit effort="0" lower="${radians(-90)}" upper="${radians(150)}" velocity="${radians(175)}"/>
-    </joint>
-    <joint type="revolute" name="${prefix}joint_3">
+      <limit
+        effort="${joint_limits['joint_2']['max_effort']}"
+        lower="${joint_limits['joint_2']['min_position']}"
+        upper="${joint_limits['joint_2']['max_position']}"
+        velocity="${joint_limits['joint_2']['max_velocity']}"/>
+    </joint>
+    <joint name="${prefix}joint_3" type="revolute">
       <origin xyz="0 0 1.095" rpy="0 0 0"/>
       <axis xyz="0 1 0"/>
       <parent link="${prefix}link_2"/>
       <child link="${prefix}link_3"/>
-      <limit effort="0" lower="${radians(-180)}" upper="${radians(75)}" velocity="${radians(175)}"/>
-    </joint>
-    <joint type="revolute" name="${prefix}joint_4">
+      <limit
+        effort="${joint_limits['joint_3']['max_effort']}"
+        lower="${joint_limits['joint_3']['min_position']}"
+        upper="${joint_limits['joint_3']['max_position']}"
+        velocity="${joint_limits['joint_3']['max_velocity']}"/>
+    </joint>
+    <joint name="${prefix}joint_4" type="revolute">
       <origin xyz="0 0 0.175" rpy="0 0 0"/>
       <axis xyz="1 0 0"/>
       <parent link="${prefix}link_3"/>
       <child link="${prefix}link_4"/>
-      <limit effort="0" lower="${radians(-400)}" upper="${radians(400)}" velocity="${radians(250)}"/>
-    </joint>
-    <joint type="revolute" name="${prefix}joint_5">
+      <limit
+        effort="${joint_limits['joint_4']['max_effort']}"
+        lower="${joint_limits['joint_4']['min_position']}"
+        upper="${joint_limits['joint_4']['max_position']}"
+        velocity="${joint_limits['joint_4']['max_velocity']}"/>
+    </joint>
+    <joint name="${prefix}joint_5" type="revolute">
       <origin xyz="1.270 0 0" rpy="0 0 0"/>
       <axis xyz="0 1 0"/>
       <parent link="${prefix}link_4"/>
       <child link="${prefix}link_5"/>
-      <limit effort="0" lower="${radians(-125)}" upper="${radians(120)}" velocity="${radians(250)}"/>
-    </joint>
-    <joint type="revolute" name="${prefix}joint_6">
+      <limit
+        effort="${joint_limits['joint_5']['max_effort']}"
+        lower="${joint_limits['joint_5']['min_position']}"
+        upper="${joint_limits['joint_5']['max_position']}"
+        velocity="${joint_limits['joint_5']['max_velocity']}"/>
+    </joint>
+    <joint name="${prefix}joint_6" type="revolute">
       <origin xyz="0 0 0" rpy="0 0 0"/>
       <axis xyz="1 0 0"/>
       <parent link="${prefix}link_5"/>
       <child link="${prefix}link_6"/>
-      <limit effort="0" lower="${radians(-400)}" upper="${radians(400)}" velocity="${radians(360)}"/>
+      <limit
+        effort="${joint_limits['joint_6']['max_effort']}"
+        lower="${joint_limits['joint_6']['min_position']}"
+        upper="${joint_limits['joint_6']['max_position']}"
+        velocity="${joint_limits['joint_6']['max_velocity']}"/>
     </joint>
     <!-- end of joint list -->
-    <!-- 'base' frame: base_link to ABB World Coordinates transform  -->
+    <!-- 'base' frame - base_link to ABB World Coordinates transform  -->
     <link name="${prefix}base" />
     <joint name="${prefix}base_link-base" type="fixed">
@@ -159,5 +189,5 @@
       <child link="${prefix}base"/>
     </joint>
-    <!-- ROS-Industrial 'flange' frame: attachment point for EEF models -->
+    <!-- ROS-Industrial 'flange' frame - attachment point for EEF models -->
     <link name="${prefix}flange"/>
     <joint type="fixed" name="${prefix}joint_6-flange">
@@ -166,5 +196,5 @@
       <child link="${prefix}flange"/>
     </joint>
-    <!-- ROS-Industrial 'tool0' frame: all-zeros tool frame -->
+    <!-- ROS-Industrial 'tool0' frame - all-zeros tool frame -->
     <link name="${prefix}tool0" />
     <joint name="${prefix}link_6-tool0" type="fixed">
