Commit message: use initial_positions.yaml in ros2 control xacro

File: urdf/abb_irb4600_40_255.ros2_control.xacro (robot description, xacro)
@@ -1,9 +1,9 @@
 <?xml version="1.0"?>
 <robot xmlns:xacro="http://www.ros.org/wiki/xacro">
-  <xacro:macro name="abb_irb_4600_ros2_control" params="
+  <xacro:macro name="abb_irb4600_ros2_control" params="
     prefix
     use_mock_hardware:=true
-    initial_positions_file:='$(find abb_irb4600_description)/config/initial_positions.yaml'
-    joint_limits_file:='$(find abb_irb4600_description)/config/joint_limits.yaml'
+    initial_positions_file
+    joint_limits_file
   ">
     <xacro:property

File: urdf/abb_irb4600_40_255.xacro (robot description, xacro)
@@ -29,6 +29,5 @@
   <xacro:include filename="$(find abb_irb4600_description)/urdf/abb_irb4600_40_255_macro.xacro"/>
   <xacro:abb_irb4600_40_255 prefix="$(arg prefix)"
-    initial_positions_file="$(arg initial_positions_file)"
-    joint_limits_parameters_file="$(arg joint_limits_file)"/>
+    joint_limits_file="$(arg joint_limits_file)"/>
   <!-- 'world' frame - default pose reference frame -->
   <link name="world" />
@@ -42,6 +41,8 @@
     <xacro:include
       filename="$(find abb_irb4600_description)/urdf/abb_irb4600_40_255.ros2_control.xacro"/>
-    <xacro:abb_irb_4600_ros2_control prefix="$(arg prefix)"
-      use_mock_hardware="$(arg use_mock_hardware)"/>
+    <xacro:abb_irb4600_ros2_control prefix="$(arg prefix)"
+      use_mock_hardware="$(arg use_mock_hardware)"
+      initial_positions_file="$(arg initial_positions_file)"
+      joint_limits_file="$(arg joint_limits_file)"/>
   </xacro:if>
 </robot>

File: urdf/abb_irb4600_40_255_macro.xacro (robot description, xacro)
@@ -23,8 +23,7 @@
   <xacro:macro name="abb_irb4600_40_255" params="
     prefix
-    initial_positions_file:='$(find abb_irb4600_description)/config/initial_positions_file.yaml'
-    joint_limits_parameters_file:='$(find abb_irb4600_description)/config/joint_limits.yaml'
+    joint_limits_file
   ">
-    <xacro:property name="joint_limits_parameters" value="${xacro.load_yaml(joint_limits_parameters_file)}"/>
+    <xacro:property name="joint_limits_parameters" value="${xacro.load_yaml(joint_limits_file)}"/>
     <xacro:property name="joint_limits" value="${joint_limits_parameters['joint_limits']}"/>
     <!-- link list -->
